File: hardware/main.brd (EAGLE design)
At the start: 49.2 x 49.5 mm, 17 parts, among them IC1 ATMEGA168-AU, J1 AVR_SPI_PRG_6NS

Commit message: Some changes to the hardware design
Parts:
- moved R3 1.27 mm to (25.4, 26.7)
- moved R7 1.27 mm to (41.9, 30.5)
- moved R8 1.27 mm to (41.9, 19.1)
- moved R6 1.27 mm to (6.35, 18.4)
- moved R9 1.27 mm to (6.35, 30.5)
- moved R5 1.27 mm to (2.22, 24.8)
- moved BATT1 1.27 mm to (24.1, 10.8)
- moved C1 1.27 mm to (8.89, 31.4)
- moved C2 1.27 mm to (11.4, 18.4)
- moved DISP2 1.27 mm to (24.1, 24.8)
- moved DOWN 1.27 mm to (24.1, 16.5)
- moved IC1 1.27 mm to (9.53, 24.8)
- moved R1 1.27 mm to (30.5, 22.9)
- moved R2 1.27 mm to (27.9, 26.7)
- moved R4 1.27 mm to (17.8, 27.3)
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Other:
- board size 49.2 x 49.5 mm -> 48.2 x 49.5 mm
